File: flipdot-interface.kicad_pcb (KiCad board)
At the start: 4 copper layers, 157 parts, among them J1 Conn_02x30_Odd_Even, Q1 BSS123, Q10 BSS123, Q11 BSS123, Q12 BSS84, Q13 BSS84, Q14 BSS84, Q15 BSS123, Q16 BSS123, Q17 BSS123, Q18 BSS84, Q19 BSS84, Q2 BSS84, Q20 BSS84, Q21 BSS123, Q22 BSS123, Q23 BSS123, Q24 BSS84, Q25 BSS84, Q26 BSS84, Q27 BSS123, Q28 BSS123, Q29 BSS123, Q3 BSS123, Q30 BSS84, Q31 BSS84, Q32 BSS84, Q33 BSS123, Q34 BSS123, Q35 BSS123, Q36 BSS84, Q37 BSS84, Q38 BSS84, Q4 BSS123, Q5 BSS123, Q6 BSS84, Q7 BSS84, Q8 BSS84, Q9 BSS123, U1 74HCT595, U10 74LVC1G19, U11 74HCT595, U12 74HCT595, U2 74HCT595, U3 74HCT595, U4 74HCT595, U5 74HCT595, U6 74HCT595, U7 ULN2803A, U8 ULN2803A, U9 ULN2803A

Commit message: moar woerk...
Parts:
- added J2: Conn_02x06_Odd_Even, Connector_IDC:IDC-Header_2x06_P2.54mm_Vertical, F.Cu at (157.5, 144.8)
- added R79: 10k, Resistor_SMD:R_0603_1608Metric, F.Cu at (147.8, 142.7)
- added R80: 10k, Resistor_SMD:R_0603_1608Metric, F.Cu at (147.8, 140.7)
- added R81: 10k, Resistor_SMD:R_0603_1608Metric, F.Cu at (147.8, 138.7)
- added R82: 10k, Resistor_SMD:R_0603_1608Metric, F.Cu at (147.8, 144.8)
Connections:
- U10 pad 3: (no net) -> /~{ROW_OE}
- U12 pad 14: (no net) -> /DI
Routing:
- net /~{ROW_OE}: track 0.00 -> 88.4 mm, vias 0 -> 2
- net /SCK: track 246.4 -> 331.7 mm, vias 10 -> 11
- net /DI: track 0.00 -> 72.8 mm, vias 0 -> 2
- net /LE: track 245.0 -> 309.8 mm, vias 10 -> 12
- net GND: track 278.5 -> 294.5 mm, vias 64 -> 67
- net /~{ROW_P_OE}: track 184.6 -> 192.1 mm
- net VCC: track 45.8 -> 47.0 mm, vias 17 -> 18
Other:
- board outline added: 99.1 x 101.6 mm

Commit message: moak woerk
Parts:
- added R83: 0R (dnp), Resistor_SMD:R_0603_1608Metric, F.Cu at (175.8, 136.9)
- added R84: 0R (dnp), Resistor_SMD:R_0603_1608Metric, F.Cu at (179.1, 136.9)
- added R85: 0R (dnp), Resistor_SMD:R_0603_1608Metric, F.Cu at (175.8, 135.1)
- added R86: 0R (dnp), Resistor_SMD:R_0603_1608Metric, F.Cu at (179.1, 135.1)
- moved C1 7.62 mm to (146.1, 125.0)
- moved C2 7.62 mm to (146.1, 94.5)
- moved C3 7.62 mm to (146.1, 64.0)
- moved D1 7.62 mm to (175.3, 63.5)
- moved D10 7.62 mm to (175.3, 116.8)
- moved D11 7.62 mm to (175.3, 74.9)
- moved D12 7.62 mm to (175.3, 97.8)
- moved D13 7.62 mm to (175.3, 120.7)
- moved D14 7.62 mm to (175.3, 78.7)
- moved D15 7.62 mm to (175.3, 101.6)
- moved D16 7.62 mm to (175.3, 124.5)
- moved D17 7.62 mm to (175.3, 82.5)
- moved D18 7.62 mm to (175.3, 105.4)
- moved D19 7.62 mm to (175.3, 128.3)
- moved D2 7.62 mm to (175.3, 86.4)
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Connections:
- J1 pad 42: (no net) -> /J1_P42
- J1 pad 43: (no net) -> /J1_P43
Routing:
- net /J1_P42: track 0.00 -> 42.2 mm, vias 0 -> 2
- net /J1_P43: track 0.00 -> 31.8 mm, vias 0 -> 2
- net VS: track 184.7 -> 163.8 mm, vias 45 -> 42
- net /Row Drivers Positive/ROW_P18: track 72.5 -> 61.3 mm, vias 2 -> 0
- net /Row Drivers Positive/ROW_P17: track 73.2 -> 62.1 mm, vias 2 -> 0
- net /Row Drivers Positive/ROW_P16: track 67.5 -> 56.7 mm, vias 2 -> 0
- net /Row Drivers Positive/ROW_P15: track 68.1 -> 57.4 mm, vias 2 -> 0
- net GND: track 294.5 -> 283.8 mm, vias 67 -> 65
- net /Row Drivers Positive/ROW_P14: track 62.4 -> 52.0 mm, vias 2 -> 0
- net /Row Drivers Positive/ROW_P13: track 63.0 -> 52.8 mm, vias 2 -> 0
- net /Row Drivers Positive/ROW_P12: track 57.4 -> 47.4 mm, vias 2 -> 0
- net /Row Drivers Positive/ROW_P11: track 58.0 -> 48.2 mm, vias 2 -> 0
- net /Row Drivers Positive/ROW_P9: track 52.9 -> 43.4 mm, vias 2 -> 0
- net /Row Drivers Positive/ROW_P10: track 52.2 -> 42.8 mm, vias 2 -> 0
- net /ROW_DI: track 160.0 -> 150.6 mm
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Other:
- board text added: "#19=P18"
- board text added: "#1=P0"
- board text added: "#21=N0"
- board text added: "#39=N18"
- board text added: "#43,VS"
- board text added: "74HCT595 #1"
- board text added: "74HCT595 #2"
- board text added: "74HCT595 #3"
- board text added: "74HCT595 #4"
- board text added: "74HCT595 #5"
- board text added: "A1,A2"
- board text added: "B0,B1"
- board text added: "D,A0"
- board text added: "J1#42"
- board text added: "J1#43"
- board text added: "MOD0,1"
- board text added: "MOD2,3"
- board text added: "MOD4,5"
- board text added: "MOD6,7"
- board text added: "N0"
- board text added: "N15"
- board text added: "N16"
- board text added: "N7"
- board text added: "N8"
- board text added: "P0"
- board text added: "P1"
- board text added: "P10"
- board text added: "P11"
- board text added: "P12"
- board text added: "P13"
- board text added: "P14"
- board text added: "P15"
- board text added: "P16"
- board text added: "P17"
- board text added: "P18"
- board text added: "P2"
- board text added: "P3"
- board text added: "P4"
- board text added: "P5"
- board text added: "P6"
- board text added: "P7"
- board text added: "P8"
- board text added: "P9"
- board text added: "Shiftreg order: #1, #2, 2x parallel { #3, #4, #5 }"
- board text added: "ULN2803A"
- board text added: "ULN2803A bases pulldowns"
- board text added: "Vcc"
- board text added: "Vcc,⏚"
- board text added: "Vs"
- board text added: "nCh"
- board text added: "negative drivers"
- board text added: "pCh"
- board text added: "positive drivers"
- board text added: "← N_G16..18"
- board text added: "↑ N_G8..15"
- board text added: "↓ N_G0..7"
- board text added: "⏚,#42"

Commit message: moar woerk
Parts:
- added C10: 100n, Capacitor_SMD:C_0603_1608Metric, F.Cu at (167.8, 127.1)
- added C11: 100n, Capacitor_SMD:C_0603_1608Metric, F.Cu at (216.7, 79.0)
- added C12: 10u, Capacitor_Tantalum_SMD:CP_EIA-3216-18_Kemet-A, F.Cu at (216.7, 81.3)
- added C13: 100n, Capacitor_SMD:C_0603_1608Metric, F.Cu at (212.6, 74.9)
- added C14: 100n, Capacitor_SMD:C_0603_1608Metric, F.Cu at (220.5, 73.7)
- added C15: 10u, Capacitor_Tantalum_SMD:CP_EIA-3216-18_Kemet-A, F.Cu at (221.5, 81.3)
- added D20: SOT23 A-C-K, Package_TO_SOT_SMD:SOT-23, F.Cu at (208.5, 74.9)
- added D21: SS1P3L, Diode_SMD:D_SMF, F.Cu at (217.2, 76.5)
- added D22: LED, LED_SMD:LED_0603_1608Metric, F.Cu at (221.0, 86.8)
- added D23: LED, LED_SMD:LED_0603_1608Metric, F.Cu at (221.0, 88.9)
- added J3: Screw_Terminal_01x04, TerminalBlock_MetzConnect:TerminalBlock_MetzConnect_Type086_RT03404HBLC_1x04_P3.81mm_Horizontal, F.Cu at (215.9, 62.2)
- added L1: L_Small, Inductor_SMD:L_Coilcraft_XxL4020, F.Cu at (217.2, 72.9)
- added R87: 68R, Resistor_SMD:R_0603_1608Metric, F.Cu at (163.3, 125.5)
- added R88: 68R, Resistor_SMD:R_0603_1608Metric, F.Cu at (163.3, 123.7)
- added R89: 68R, Resistor_SMD:R_0603_1608Metric, F.Cu at (163.3, 121.9)
- added R91: 10k, Resistor_SMD:R_0603_1608Metric, F.Cu at (212.6, 80.5)
- added R92: 150k, Resistor_SMD:R_0603_1608Metric, F.Cu at (207.3, 78.5)
- added R93: 10k, Resistor_SMD:R_0603_1608Metric, F.Cu at (209.3, 78.5)
- added R94: 1k, Resistor_SMD:R_0603_1608Metric, F.Cu at (217.6, 86.8)
- added R95: 1k, Resistor_SMD:R_0603_1608Metric, F.Cu at (217.6, 88.9)
- added R96: 10k, Resistor_SMD:R_0603_1608Metric, F.Cu at (176.0, 119.4)
- added R97: 10k, Resistor_SMD:R_0603_1608Metric, F.Cu at (176.0, 124.7)
- added R98: 10k, Resistor_SMD:R_0603_1608Metric, F.Cu at (176.0, 122.9)
- added R99: 10k, Resistor_SMD:R_0603_1608Metric, F.Cu at (176.0, 121.2)
- added U13: 74HCT244, Package_SO:SSOP-20_4.4x6.5mm_P0.65mm, F.Cu at (169.9, 122.4)
- added U14: LM2734Y, Package_TO_SOT_SMD:TSOT-23-6, F.Cu at (212.6, 77.7)
- moved C1 90.0 mm to (195.6, 49.8)
- moved R58 83.0 mm to (197.4, 49.8), turned to -90 degrees
- moved R59 82.5 mm to (135.9, 108.5), turned to 90 degrees
- moved C4 82.1 mm to (135.9, 104.6), turned to 90 degrees
- moved U4 77.1 mm to (142.2, 106.7), turned to 90 degrees
- moved C5 67.1 mm to (156.5, 104.6), turned to 90 degrees
- moved J2 66.7 mm to (221.0, 124.5), turned to 180 degrees
- moved C9 65.4 mm to (141.7, 115.6)
- moved U12 65.3 mm to (139.7, 121.9)
- moved J1 64.8 mm to (127.0, 50.8)
- moved R77 64.7 mm to (152.4, 88.6), turned to 0 degrees
- moved R12 64.3 mm to (136.7, 83.8)
- moved R75 63.6 mm to (152.4, 90.4), turned to 0 degrees
- moved U7 62.6 mm to (142.2, 94.0), turned to 180 degrees
- moved R73 62.5 mm to (152.4, 92.2), turned to 0 degrees
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Connections:
- J2 pad 1: /DI -> /DI_LV
- J2 pad 2: /SCK -> /SCK_LV
- J2 pad 3: /LE -> /LE_LV
- J2 pad 4: /~{ROW_OE} -> /~{ROW_OE}_LV
- R60 pad 1: /Row Drivers Negative/ROW_N_G0 -> /Row Drivers Negative/ROW_N_G7
- R61 pad 1: /Row Drivers Negative/ROW_N_G8 -> /Row Drivers Negative/ROW_N_G15
- R62 pad 1: /Row Drivers Negative/ROW_N_G16 -> /Row Drivers Negative/ROW_N_G18
- R63 pad 1: /Row Drivers Negative/ROW_N_G1 -> /Row Drivers Negative/ROW_N_G6
- R64 pad 1: /Row Drivers Negative/ROW_N_G9 -> /Row Drivers Negative/ROW_N_G14
- R66 pad 1: /Row Drivers Negative/ROW_N_G2 -> /Row Drivers Negative/ROW_N_G5
- R67 pad 1: /Row Drivers Negative/ROW_N_G10 -> /Row Drivers Negative/ROW_N_G13
- R68 pad 1: /Row Drivers Negative/ROW_N_G18 -> /Row Drivers Negative/ROW_N_G16
- R69 pad 1: /Row Drivers Negative/ROW_N_G3 -> /Row Drivers Negative/ROW_N_G4
- R70 pad 1: /Row Drivers Negative/ROW_N_G11 -> /Row Drivers Negative/ROW_N_G12
- R71 pad 1: /Row Drivers Negative/ROW_N_G4 -> /Row Drivers Negative/ROW_N_G3
- R72 pad 1: /Row Drivers Negative/ROW_N_G12 -> /Row Drivers Negative/ROW_N_G11
- R73 pad 1: /Row Drivers Negative/ROW_N_G5 -> /Row Drivers Negative/ROW_N_G2
- R74 pad 1: /Row Drivers Negative/ROW_N_G13 -> /Row Drivers Negative/ROW_N_G10
- R75 pad 1: /Row Drivers Negative/ROW_N_G6 -> /Row Drivers Negative/ROW_N_G1
- R76 pad 1: /Row Drivers Negative/ROW_N_G14 -> /Row Drivers Negative/ROW_N_G9
- R77 pad 1: /Row Drivers Negative/ROW_N_G7 -> /Row Drivers Negative/ROW_N_G0
- R78 pad 1: /Row Drivers Negative/ROW_N_G15 -> /Row Drivers Negative/ROW_N_G8
- U7 pad 1: /Row Drivers Negative/ROW_N_G0 -> /Row Drivers Negative/ROW_N_G7
- U7 pad 11: /Row Drivers Negative/ROW_N7 -> /Row Drivers Negative/ROW_N0
- U7 pad 12: /Row Drivers Negative/ROW_N6 -> /Row Drivers Negative/ROW_N1
- U7 pad 13: /Row Drivers Negative/ROW_N5 -> /Row Drivers Negative/ROW_N2
- U7 pad 14: /Row Drivers Negative/ROW_N4 -> /Row Drivers Negative/ROW_N3
- U7 pad 15: /Row Drivers Negative/ROW_N3 -> /Row Drivers Negative/ROW_N4
- U7 pad 16: /Row Drivers Negative/ROW_N2 -> /Row Drivers Negative/ROW_N5
- U7 pad 17: /Row Drivers Negative/ROW_N1 -> /Row Drivers Negative/ROW_N6
- U7 pad 18: /Row Drivers Negative/ROW_N0 -> /Row Drivers Negative/ROW_N7
- U7 pad 2: /Row Drivers Negative/ROW_N_G1 -> /Row Drivers Negative/ROW_N_G6
- U7 pad 3: /Row Drivers Negative/ROW_N_G2 -> /Row Drivers Negative/ROW_N_G5
- U7 pad 4: /Row Drivers Negative/ROW_N_G3 -> /Row Drivers Negative/ROW_N_G4
- U7 pad 5: /Row Drivers Negative/ROW_N_G4 -> /Row Drivers Negative/ROW_N_G3
- U7 pad 6: /Row Drivers Negative/ROW_N_G5 -> /Row Drivers Negative/ROW_N_G2
- U7 pad 7: /Row Drivers Negative/ROW_N_G6 -> /Row Drivers Negative/ROW_N_G1
- U7 pad 8: /Row Drivers Negative/ROW_N_G7 -> /Row Drivers Negative/ROW_N_G0
- U8 pad 1: /Row Drivers Negative/ROW_N_G8 -> /Row Drivers Negative/ROW_N_G15
- U8 pad 11: /Row Drivers Negative/ROW_N15 -> /Row Drivers Negative/ROW_N8
- U8 pad 12: /Row Drivers Negative/ROW_N14 -> /Row Drivers Negative/ROW_N9
- U8 pad 13: /Row Drivers Negative/ROW_N13 -> /Row Drivers Negative/ROW_N10
- U8 pad 14: /Row Drivers Negative/ROW_N12 -> /Row Drivers Negative/ROW_N11
- U8 pad 15: /Row Drivers Negative/ROW_N11 -> /Row Drivers Negative/ROW_N12
- U8 pad 16: /Row Drivers Negative/ROW_N10 -> /Row Drivers Negative/ROW_N13
- U8 pad 17: /Row Drivers Negative/ROW_N9 -> /Row Drivers Negative/ROW_N14
- U8 pad 18: /Row Drivers Negative/ROW_N8 -> /Row Drivers Negative/ROW_N15
- U8 pad 2: /Row Drivers Negative/ROW_N_G9 -> /Row Drivers Negative/ROW_N_G14
- U8 pad 3: /Row Drivers Negative/ROW_N_G10 -> /Row Drivers Negative/ROW_N_G13
- U8 pad 4: /Row Drivers Negative/ROW_N_G11 -> /Row Drivers Negative/ROW_N_G12
- U8 pad 5: /Row Drivers Negative/ROW_N_G12 -> /Row Drivers Negative/ROW_N_G11
- U8 pad 6: /Row Drivers Negative/ROW_N_G13 -> /Row Drivers Negative/ROW_N_G10
- U8 pad 7: /Row Drivers Negative/ROW_N_G14 -> /Row Drivers Negative/ROW_N_G9
- U8 pad 8: /Row Drivers Negative/ROW_N_G15 -> /Row Drivers Negative/ROW_N_G8
- U9 pad 1: /Row Drivers Negative/ROW_N_G16 -> (no net)
- U9 pad 11: (no net) -> /Row Drivers Negative/ROW_N16
- U9 pad 12: (no net) -> /Row Drivers Negative/ROW_N17
- U9 pad 13: (no net) -> /Row Drivers Negative/ROW_N18
- U9 pad 16: /Row Drivers Negative/ROW_N18 -> (no net)
- U9 pad 17: /Row Drivers Negative/ROW_N17 -> (no net)
- U9 pad 18: /Row Drivers Negative/ROW_N16 -> (no net)
- U9 pad 2: /Row Drivers Negative/ROW_N_G17 -> (no net)
- U9 pad 3: /Row Drivers Negative/ROW_N_G18 -> (no net)
- U9 pad 4: GND -> (no net)
- U9 pad 5: GND -> (no net)
- U9 pad 6: GND -> /Row Drivers Negative/ROW_N_G18
- U9 pad 7: GND -> /Row Drivers Negative/ROW_N_G17
- U9 pad 8: GND -> /Row Drivers Negative/ROW_N_G16
Routing:
- net VS: track 163.8 -> 263.8 mm, vias 42 -> 26
- net /~{ROW_OE}_LV: track 0.00 -> 92.7 mm
- net /SCK_LV: track 0.00 -> 82.5 mm
- net /~{ROW_OE}: track 88.4 -> 14.1 mm, vias 2 -> 0
- net /LE_LV: track 0.00 -> 72.8 mm
- net /DI_LV: track 0.00 -> 67.7 mm
- net /~{ROW_P_OE}: track 184.1 -> 133.9 mm, vias 6 -> 2
- net /DI: track 72.8 -> 24.2 mm
- net /SCK: track 323.7 -> 276.1 mm, vias 11 -> 6
- net /Row Drivers Negative/ROW_N17: track 17.2 -> 54.6 mm, vias 0 -> 1
- net /Row Drivers Negative/ROW_N16: track 21.1 -> 57.6 mm, vias 0 -> 1
- net /Row Drivers Negative/ROW_N18: track 20.2 -> 56.2 mm, vias 0 -> 1
- net Net-(U1-Pad9): track 43.3 -> 8.59 mm
- net Net-(U2-Pad9): track 42.6 -> 8.34 mm
- net /Row Drivers Positive/ROW_P18: track 61.3 -> 31.1 mm
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Other:
- board size 99.1 x 101.6 mm -> 109.2 x 88.9 mm
- board text added: "DI"
- board text added: "N0 ... N7"
- board text added: "N16 N17 N18"
- board text added: "N8 ... N15"
- board text added: "SCK LE"
- board text added: "SCK LE DI"
- board text added: "VS"
- board text added: "~{OE}"
- board text added: "~{ROW_N_OE}"
- board text added: "~{ROW_P_OE}"
- board text added: "⏚"
- board text removed: "74HCT595 #1"
- board text removed: "74HCT595 #2"
- board text removed: "74HCT595 #3"
- board text removed: "74HCT595 #4"
- board text removed: "74HCT595 #5"
- board text removed: "N0"
- board text removed: "N15"
- board text removed: "N16"
- board text removed: "N7"
- board text removed: "N8"
- board text removed: "Shiftreg order: #1, #2, 2x parallel { #3, #4, #5 }"
- board text removed: "ULN2803A"
- board text removed: "ULN2803A bases pulldowns"
- board text removed: "nCh"
- board text removed: "negative drivers"
- board text removed: "pCh"
- board text removed: "positive drivers"
- board text removed: "← N_G16..18"
- board text removed: "↑ N_G8..15"
- board text removed: "↓ N_G0..7"

Commit message: moar woerk
Parts:
- moved R83 5.99 mm to (140.8, 113.3)
- moved R85 5.98 mm to (140.8, 111.6)
- moved R84 5.86 mm to (144.0, 113.3)
- moved R86 5.85 mm to (144.0, 111.6)
Routing:
- net /J1_P43: track 17.1 -> 24.8 mm
- net /J1_P42: track 28.6 -> 34.6 mm
- net VCC: track 72.4 -> 67.3 mm
- net VS: track 263.8 -> 268.9 mm, vias 26 -> 27
- net /COL_B0: track 32.7 -> 27.9 mm
- net /COL_B1: track 31.1 -> 27.7 mm
- net /COL_A1: track 28.3 -> 25.7 mm
- net /COL_A2: track 28.2 -> 26.7 mm
- net /COL_D: track 49.8 -> 49.0 mm

Commit message: more work
Parts:
- removed C9: 100n, Capacitor_SMD:C_0603_1608Metric
- added J4: Conn_02x06_Odd_Even, Connector_IDC:IDC-Header_2x06_P2.54mm_Vertical, F.Cu at (199.4, 112.5)
- added JP1: SolderJumper_2_Bridged, Jumper:SolderJumper-2_P1.3mm_Bridged_Pad1.0x1.5mm, B.Cu at (135.4, 113.3)
- added JP2: SolderJumper_2_Bridged, Jumper:SolderJumper-2_P1.3mm_Bridged_Pad1.0x1.5mm, B.Cu at (135.4, 116.1)
- added JP3: SolderJumper_2_Bridged, Jumper:SolderJumper-2_P1.3mm_Bridged_Pad1.0x1.5mm, B.Cu at (135.4, 118.9)
- added JP4: SolderJumper_2_Bridged, Jumper:SolderJumper-2_P1.3mm_Bridged_Pad1.0x1.5mm, B.Cu at (135.4, 121.7)
- added JP5: SolderJumper_2_Bridged, Jumper:SolderJumper-2_P1.3mm_Bridged_Pad1.0x1.5mm, B.Cu at (135.4, 124.5)
- added JP6: SolderJumper_2_Bridged, Jumper:SolderJumper-2_P1.3mm_Bridged_Pad1.0x1.5mm, B.Cu at (135.4, 127.0)
- added R100: 68R, Resistor_SMD:R_0603_1608Metric, F.Cu at (159.8, 112.3)
- added R101: 68R, Resistor_SMD:R_0603_1608Metric, F.Cu at (186.9, 124.5)
- added R102: 68R, Resistor_SMD:R_0603_1608Metric, F.Cu at (186.9, 122.7)
- added R103: 68R, Resistor_SMD:R_0603_1608Metric, F.Cu at (186.9, 120.9)
- added R104: 68R, Resistor_SMD:R_0603_1608Metric, F.Cu at (186.9, 119.1)
- added R105: 0R (dnp), Resistor_SMD:R_0603_1608Metric, F.Cu at (173.5, 115.8)
- added R106: 0R (dnp), Resistor_SMD:R_0603_1608Metric, F.Cu at (171.7, 115.8)
- added R107: 0R (dnp), Resistor_SMD:R_0603_1608Metric, F.Cu at (211.1, 104.4)
- added R108: 0R (dnp), Resistor_SMD:R_0603_1608Metric, F.Cu at (190.8, 128.0)
- added R90: 68R, Resistor_SMD:R_0603_1608Metric, F.Cu at (159.8, 114.0)
- U12: value 74HCT595 -> ULN2803A; footprint Package_SO:SOIC-16_3.9x9.9mm_P1.27mm -> Package_SO:SOIC-18W_7.5x11.6mm_P1.27mm
- moved J2 21.6 mm to (199.4, 125.2), turned to 90 degrees
- moved R80 18.9 mm to (163.8, 123.2)
- moved R82 16.3 mm to (162.1, 119.9), turned to 90 degrees
- moved R79 15.3 mm to (162.1, 123.2)
- moved R81 9.72 mm to (167.5, 113.2)
- moved C8 9.33 mm to (163.4, 113.2), turned to 90 degrees
- moved C7 6.84 mm to (157.0, 115.8)
- moved R96 4.83 mm to (180.8, 119.1)
- moved R97 4.83 mm to (180.8, 124.5)
- moved R98 4.83 mm to (180.8, 122.7)
- moved R99 4.83 mm to (180.8, 120.9)
- moved C10 4.38 mm to (172.1, 126.4)
- moved U13 4.38 mm to (174.2, 121.7)
- moved R87 4.20 mm to (167.1, 123.7)
- moved R89 4.20 mm to (167.1, 120.1)
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Connections:
- net Net-(R89-Pad1) renamed /DI_x
- C13 pad 2: /VREG_BOOST -> Net-(C13-Pad2)
- D20 pad 3: /VREG_BOOST -> Net-(C13-Pad2)
- J2 pad 11: (no net) -> Net-(J2-Pad11)
- J2 pad 12: (no net) -> Net-(J2-Pad11)
- J2 pad 5: (no net) -> Net-(J2-Pad5)
- R87 pad 2: /DI -> /SCK
- R89 pad 2: /SCK -> /DI
- R97 pad 1: /DI_LV -> /SCK_LV
- R99 pad 1: /SCK_LV -> /DI_LV
- U10 pad 1: /COL_D -> /COL_D_LV
- U10 pad 4: /~{ROW_N_OE} -> Net-(U10-Pad4)
- U10 pad 6: /~{ROW_P_OE} -> Net-(U10-Pad6)
- U11 pad 1: /COL_A1 -> Net-(U12-Pad7)
- U11 pad 14: Net-(U11-Pad14) -> /DI
- U11 pad 15: /COL_A0 -> Net-(U12-Pad8)
- U11 pad 2: /COL_A2 -> Net-(U12-Pad6)
- U11 pad 3: /COL_B0 -> Net-(U12-Pad5)
- U11 pad 4: /COL_B1 -> Net-(U12-Pad4)
- U11 pad 5: /COL_D -> /COL_D_LV
- U11 pad 6: (no net) -> Net-(U11-Pad6)
- U11 pad 7: (no net) -> Net-(U11-Pad7)
- U12 pad 1: /MODULE_A1 -> Net-(U11-Pad7)
- U12 pad 10: VCC -> VS
- U12 pad 11: /SCK -> /COL_A0
- U12 pad 12: /LE -> /COL_A1
- U12 pad 13: GND -> /COL_A2
- U12 pad 14: /DI -> /COL_B0
- U12 pad 15: /MODULE_A0 -> /COL_B1
- U12 pad 16: VCC -> /COL_D
- U12 pad 2: /MODULE_A2 -> Net-(U11-Pad6)
- U12 pad 3: /MODULE_A3 -> /COL_D_LV
- U12 pad 4: /MODULE_A4 -> Net-(U12-Pad4)
- U12 pad 5: /MODULE_A5 -> Net-(U12-Pad5)
- U12 pad 6: /MODULE_A6 -> Net-(U12-Pad6)
- U12 pad 7: /MODULE_A7 -> Net-(U12-Pad7)
- U12 pad 8: GND -> Net-(U12-Pad8)
- U12 pad 9: Net-(U11-Pad14) -> GND
- U13 pad 11: GND -> /~{ROW_OE}
- U13 pad 13: GND -> /DO_LV_SEL
- U13 pad 15: GND -> /LE
- U13 pad 17: GND -> /SCK
- U13 pad 2: /DI_LV -> /SCK_LV
- U13 pad 3: (no net) -> Net-(U13-Pad3)
- U13 pad 5: (no net) -> Net-(U13-Pad5)
- U13 pad 6: /SCK_LV -> /DI_LV
- U13 pad 7: (no net) -> Net-(U13-Pad7)
- U13 pad 9: (no net) -> Net-(U13-Pad9)
- U14 pad 1: /VREG_BOOST -> (no net)
- U3 pad 9: (no net) -> /DO_P
Routing:
- net /DO_P: track 0.00 -> 58.4 mm, vias 0 -> 2
- net /~{ROW_OE}_LV: track 92.7 -> 36.8 mm
- net /SCK_LV: track 82.5 -> 34.8 mm
- net /LE_LV: track 72.8 -> 28.4 mm
- net /DI_LV: track 67.7 -> 29.0 mm
- net /~{ROW_OE}_OUT: track 0.00 -> 34.2 mm
- net /DO: track 0.00 -> 33.5 mm, vias 0 -> 2
- net /SCK_OUT: track 0.00 -> 32.4 mm
- net /COL_D_LV: track 0.00 -> 29.5 mm, vias 0 -> 2
- net Net-(U11-Pad14): track 28.8 -> 0.00 mm, vias 2 -> 0
- net /SCK: track 276.1 -> 302.1 mm
- net /LE_OUT: track 0.00 -> 25.3 mm
- net /COL_D: track 49.0 -> 27.3 mm, vias 2 -> 0
- net /LE: track 282.7 -> 304.0 mm
- net Net-(J2-Pad11): track 0.00 -> 20.9 mm
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Other:
- board text added: "A0 A1 A2 B0 B1 D Mod0 Mod1"
- board text added: "A7, A6, A5, A4, A3, A2"
- board text added: "DI LE SCK"
- board text added: "DO"
- board text added: "DO #5"
- board text added: "DO LE SCK"
- board text added: "Input"
- board text added: "LE SCK"
- board text added: "N_~{OE}"
- board text added: "Output"
- board text added: "P_~{OE}"
- board text added: "SCK ~{OE} - - ⏚ (Vcc) DI LE (DO) - ⏚ (Vcc)"
- board text added: "SCK ~{OE} - - ⏚ (Vcc) DO LE - - ⏚ (Vcc)"
- board text added: "Vcc #11/#12"
- board text added: "chain"
- board text added: "input pullup/dn"
- board text added: "n-Ch"
- board text added: "output series term"
- board text added: "p-Ch"
- board text added: "parallel"
- board text added: "positive driver"
- board text added: "pulldn"
- board text removed: "SCK LE"
- board text removed: "SCK LE DI"

Commit message: More work, moved digital stuff to sub-schematic.
Parts:
- removed R80, R81, R82: 10k, Resistor_SMD:R_0603_1608Metric
- added C16: 10u, Capacitor_Tantalum_SMD:CP_EIA-3216-18_Kemet-A, F.Cu at (201.7, 79.2)
- added C17: 100n, Capacitor_SMD:C_0603_1608Metric, F.Cu at (206.8, 77.2)
- added C18: 10u, Capacitor_Tantalum_SMD:CP_EIA-3216-18_Kemet-A, F.Cu at (206.8, 79.2)
- added C9: 100n, Capacitor_SMD:C_0603_1608Metric, F.Cu at (201.7, 77.2)
- added D24: LED, LED_SMD:LED_0603_1608Metric, F.Cu at (218.1, 70.6)
- added U15: AP1117-33, Package_TO_SOT_SMD:SOT-223-3_TabPin2, F.Cu at (204.7, 72.6)
- R79: value 10k -> 1k
- moved R79 74.4 mm to (214.6, 70.6), turned to 0 degrees
- moved D20 22.5 mm to (199.7, 54.2), turned to -90 degrees
- moved C13 21.9 mm to (199.9, 57.1)
- moved C11 21.9 mm to (203.9, 61.2)
- moved C12 21.9 mm to (203.9, 63.5)
- moved U14 21.9 mm to (199.9, 59.9)
- moved C14 21.9 mm to (207.7, 55.9)
- moved C15 21.9 mm to (208.7, 63.5)
- moved D21 21.9 mm to (204.4, 58.7)
- moved L1 21.9 mm to (204.4, 55.1)
- moved R94 20.5 mm to (214.7, 66.5)
- moved R95 20.5 mm to (214.7, 68.6)
- moved D22 20.5 mm to (218.1, 66.5)
- moved D23 20.5 mm to (218.1, 68.6)
- moved R93 18.8 mm to (199.4, 62.5), turned to 180 degrees
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Connections:
- net /COL_D_LV renamed /Digital Pin Drivers/COL_D_LV
- C13 pad 2: Net-(C13-Pad2) -> /VREG_BOOST
- D20 pad 3: Net-(C13-Pad2) -> /VREG_BOOST
- R79 pad 1: /LE -> +3V3
- R79 pad 2: GND -> Net-(D24-Pad2)
- U14 pad 1: (no net) -> /VREG_BOOST
Routing:
- net +3V3: track 0.00 -> 20.8 mm
- net VS: track 276.4 -> 263.7 mm
- net Net-(C13-Pad2): track 4.35 -> 0.00 mm
- net /VREG_BOOST: track 0.00 -> 4.21 mm
- net Net-(R91-Pad2): track 1.97 -> 5.23 mm
- net VCC: track 65.7 -> 68.8 mm, vias 22 -> 25
- net GND: track 280.8 -> 283.0 mm, vias 84 -> 89
- net /SCK: track 302.1 -> 301.0 mm
- net /VREG_FB: track 4.46 -> 3.43 mm
Other:
- board text removed: "DI"
- board text removed: "LE SCK"
- board text removed: "pulldn"
