File: drv_pos.kicad_sch (KiCad schematic)
At the start: 121 parts, among them Q1 BSS123, Q10 BSS123, Q11 BSS123, Q12 BSS84, Q13 BSS84, Q14 BSS84, Q15 BSS123, Q16 BSS123, Q17 BSS123, Q18 BSS84, Q19 BSS84, Q2 BSS84, Q20 BSS84, Q21 BSS123, Q22 BSS123, Q23 BSS123, Q24 BSS84, Q25 BSS84, Q26 BSS84, Q27 BSS123, Q28 BSS123, Q29 BSS123, Q3 BSS123, Q30 BSS84, Q31 BSS84, Q32 BSS84, Q33 BSS123, Q34 BSS123, Q35 BSS123, Q36 BSS84, Q37 BSS84, Q38 BSS84, Q4 BSS123, Q5 BSS123, Q6 BSS84, Q7 BSS84, Q8 BSS84, Q9 BSS123, U1 74HCT595, U2 74HCT595, U3 74HCT595

Commit message: more work
Connections:
- net ROW_P_DO: now reaches U3.9 (QH')
- no-connect marks 6 -> 5
Other:
- moved on the sheet: C1, C2, C3, D4, Q5, Q8, R12, R58, R6, R9, U1, U2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

Commit message: Change positive drivers to a TLE75080-ESD, octal high side driver
Parts:
- removed D1, D10, D11, D12, D13, D14, D15, D16, D17, D18, D19, D2, D3, D4, D5, D6, D7, D8, D9: SOT23 A-C-K, Package_TO_SOT_SMD:SOT-23, symbol Device:D_Dual_Series_ACK_Parallel
- removed Q1, Q10, Q11, Q15, Q16, Q17, Q21, Q22, Q23, Q27, Q28, Q29, Q3, Q33, Q34, Q35, Q4, Q5, Q9: BSS123, Package_TO_SOT_SMD:SOT-23, symbol Transistor_FET:BSS123
- removed Q12, Q13, Q14, Q18, Q19, Q2, Q20, Q24, Q25, Q26, Q30, Q31, Q32, Q36, Q37, Q38, Q6, Q7, Q8: BSS84, Package_TO_SOT_SMD:SOT-23, symbol Transistor_FET:BSS84
- removed R1, R10, R11, R12, R13, R14, R15, R16, R17, R18, R19, R2, R20, R21, R22, R23, R24, R25, R26, R27, R28, R29, R3, R30, R31, R32, R33, R34, R35, R36, R37, R38, R39, R4, R40, R41, R42, R43, R44, R45, R46, R47, R48, R49, R5, R50, R51, R52, R53, R54, R55, R56, R57, R6, R7, R8, R9: 10k, Resistor_SMD:R_0603_1608Metric, symbol Device:R
- removed U1, U2, U3: 74HCT595, Package_SO:SOIC-16_3.9x9.9mm_P1.27mm, symbol 74xx:74HCT595
- added C19, C20, C21: 100n, Capacitor_SMD:C_0603_1608Metric, symbol Device:C_Small
- added U16, U17, U18: tle75080-esd, vogelchr_package_so:Infineon-PG-TSDSO-24-51, symbol vogelchr_ic:tle75080-esd
Connections:
- net GND: now also C19.1, C20.1, C21.1, U16.22 (IN1), U16.23 (IN0), U16.25 (GND(pad)), U16.5 (GND), U17.22 (IN1), U17.23 (IN0), U17.25 (GND(pad)), U17.5 (GND), U18.22 (IN1), U18.23 (IN0), U18.25 (GND(pad)), U18.5 (GND)
- net ROW_P0: now also U16.6 (OUT0)
- net ROW_P1: now also U16.19 (OUT1)
- net ROW_P10: now also U17.8 (OUT2)
- net ROW_P11: now also U17.17 (OUT4)
- net ROW_P12: now also U17.10 (OUT4)
- net ROW_P13: now also U17.15 (OUT5)
- net ROW_P14: now also U17.11 (OUT6)
- net ROW_P15: now also U17.14 (OUT7)
- net ROW_P16: now also U18.6 (OUT0)
- net ROW_P17: now also U18.19 (OUT1)
- net ROW_P18: now also U18.8 (OUT2)
- net ROW_P2: now also U16.8 (OUT2)
- net ROW_P3: now also U16.17 (OUT4)
- net ROW_P4: now also U16.10 (OUT4)
- net ROW_P5: now also U16.15 (OUT5)
- net ROW_P6: now also U16.11 (OUT6)
- net ROW_P7: now also U16.14 (OUT7)
- net ROW_P8: now also U17.6 (OUT0)
- net ROW_P9: now also U17.19 (OUT1)
- net ROW_P_DI: now also U16.3 (SI)
- net ROW_P_DO: now also U18.4 (SO)
- net ROW_P_SCK: now also U16.2 (SCKL), U17.2 (SCKL), U18.2 (SCKL)
- net VCC: now also C19.2, C20.2, C21.2, U16.24 (VDD), U17.24 (VDD), U18.24 (VDD); no longer C1.2, C2.2, C3.2
- net VS: now also C1.2, C2.2, C3.2, U16.16 (VS2), U16.20 (VS), U16.9 (VS1), U17.16 (VS2), U17.20 (VS), U17.9 (VS1), U18.16 (VS2), U18.20 (VS), U18.9 (VS1)
- net ~{ROW_P_OE}: now also U16.21 (IDLE), U17.21 (IDLE), U18.21 (IDLE)
- new net: U17.4 (SO), U18.3 (SI)
- new net: U16.4 (SO), U17.3 (SI)
- new net ~{ROW_P_CS}: U16.1 (~{CS}), U17.1 (~{CS}), U18.1 (~{CS})
- no-connect marks 5 -> 0
Other:
- moved on the sheet: R58

Commit message: Change negative drivers to a TLE75008-ESD, octal low side driver.
Parts:
- removed R58: 10k, Resistor_SMD:R_0603_1608Metric, symbol Device:R
Connections:
- net ~{ROW_P_OE} renamed ROW_P_IDLE
