File: flipdot-interface.kicad_sch (KiCad schematic)
At the start: 8 parts, among them J1 Conn_02x30_Odd_Even, J2 Conn_02x06_Odd_Even, U10 74LVC1G19, U11 74HCT595, U12 74HCT595

Commit message: moar woerk...
Parts:
- added R79, R80, R81, R82: 10k, Resistor_SMD:R_0603_1608Metric, symbol Device:R
- J2: footprint (none) -> Connector_IDC:IDC-Header_2x06_P2.54mm_Vertical
Connections:
- net DI: now also R82.1
- net GND: now also R79.2, R80.2, R82.2
- net LE: now also R79.1
- net SCK: now also R80.1
- net VCC: now also R81.1
- net ~{ROW_OE}: now also R81.2
- no-connect marks 4 -> 10
Other:
- moved on the sheet: C7, C8, C9, U10, U11, U12

Commit message: moak woerk
Parts:
- added R83, R84, R85, R86: 0R (dnp), Resistor_SMD:R_0603_1608Metric, symbol Device:R
Connections:
- net VCC: now also R84.1, R86.1
- net VS: now also R83.1, R85.1
- net J1_P43: now reaches J1.43 (Pin_43)
- net J1_P43: now also R85.2, R86.2
- net PULLUP renamed J1_P42
- net J1_P42: now also R83.2, R84.2
Changed lines of the file:
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@@
   (junction (at 40.64 25.4) (diameter 0) (color 0 0 0 0))
   (junction (at 41.91 22.86) (diameter 0) (color 0 0 0 0))
+  (junction (at 50.8 76.2) (diameter 0) (color 0 0 0 0))
+  (junction (at 50.8 87.63) (diameter 0) (color 0 0 0 0))
   (junction (at 163.83 48.26) (diameter 0) (color 0 0 0 0))
   (junction (at 170.18 87.63) (diameter 0) (color 0 0 0 0))
@@
     (stroke (width 0) (type default) (color 0 0 0 0))
   )
+  (wire (pts (xy 40.64 74.93) (xy 41.91 74.93))
+    (stroke (width 0) (type default) (color 0 0 0 0))
+  )
+  (wire (pts (xy 40.64 77.47) (xy 41.91 77.47))
+    (stroke (width 0) (type default) (color 0 0 0 0))
+  )
+  (wire (pts (xy 40.64 86.36) (xy 41.91 86.36))
+    (stroke (width 0) (type default) (color 0 0 0 0))
+  )
+  (wire (pts (xy 40.64 88.9) (xy 41.91 88.9))
+    (stroke (width 0) (type default) (color 0 0 0 0))
+  )
   (wire (pts (xy 41.91 22.86) (xy 45.72 22.86))
     (stroke (width 0) (type default) (color 0 0 0 0))
@@
     (stroke (width 0) (type default) (color 0 0 0 0))
   )
+  (wire (pts (xy 49.53 74.93) (xy 50.8 74.93))
+    (stroke (width 0) (type default) (color 0 0 0 0))
+  )
+  (wire (pts (xy 49.53 77.47) (xy 50.8 77.47))
+    (stroke (width 0) (type default) (color 0 0 0 0))
+  )
+  (wire (pts (xy 49.53 86.36) (xy 50.8 86.36))
+    (stroke (width 0) (type default) (color 0 0 0 0))
+  )
+  (wire (pts (xy 49.53 88.9) (xy 50.8 88.9))
+    (stroke (width 0) (type default) (color 0 0 0 0))
+  )
   (wire (pts (xy 49.53 125.73) (xy 50.8 125.73))
+    (stroke (width 0) (type default) (color 0 0 0 0))
+  )
+  (wire (pts (xy 50.8 74.93) (xy 50.8 76.2))
+    (stroke (width 0) (type default) (color 0 0 0 0))
+  )
+  (wire (pts (xy 50.8 76.2) (xy 50.8 77.47))
+    (stroke (width 0) (type default) (color 0 0 0 0))
+  )
+  (wire (pts (xy 50.8 76.2) (xy 64.77 76.2))
+    (stroke (width 0) (type default) (color 0 0 0 0))
+  )
+  (wire (pts (xy 50.8 86.36) (xy 50.8 87.63))
+    (stroke (width 0) (type default) (color 0 0 0 0))
+  )
+  (wire (pts (xy 50.8 87.63) (xy 50.8 88.9))
+    (stroke (width 0) (type default) (color 0 0 0 0))
+  )
+  (wire (pts (xy 50.8 87.63) (xy 64.77 87.63))
     (stroke (width 0) (type default) (color 0 0 0 0))
   )
@@
     (effects (font (size 1.27 1.27)) (justify left bottom))
   )
+  (label "J1_P42" (at 57.15 76.2 0)
+    (effects (font (size 1.27 1.27)) (justify left bottom))
+  )
+  (label "J1_P43" (at 57.15 87.63 0)
+    (effects (font (size 1.27 1.27)) (justify left bottom))
+  )
   (label "SCK" (at 64.77 115.57 0)
     (effects (font (size 1.27 1.27)) (justify left bottom))
@@
     (effects (font (size 1.27 1.27)) (justify left bottom))
   )
+  (label "J1_P43" (at 88.9 82.55 0)
+    (effects (font (size 1.27 1.27)) (justify left bottom))
+  )
   (label "COL_D" (at 88.9 87.63 0)
     (effects (font (size 1.27 1.27)) (justify left bottom))
@@
     (effects (font (size 1.27 1.27)) (justify left bottom))
   )
-  (label "PULLUP" (at 123.19 80.01 0)
+  (label "J1_P42" (at 123.19 80.01 0)
     (effects (font (size 1.27 1.27)) (justify left bottom))
   )
@@
   (label "ROW_DI" (at 246.38 71.12 0)
     (effects (font (size 1.27 1.27)) (justify left bottom))
+  )
+  (symbol (lib_id "power:VS") (at 40.64 74.93 90) (unit 1)
+    (in_bom yes) (on_board yes)
+    (property "Reference" "#PWR0143" (id 0) (at 44.45 80.01 0)
+      (effects (font (size 1.27 1.27)) hide)
+    )
+    (property "Value" "VS" (id 1) (at 36.83 74.93 90)
+      (effects (font (size 1.27 1.27)) (justify left))
+    )
+    (property "Footprint" "" (id 2) (at 40.64 74.93 0)
+      (effects (font (size 1.27 1.27)) hide)
+    )
+    (property "Datasheet" "" (id 3) (at 40.64 74.93 0)
+      (effects (font (size 1.27 1.27)) hide)
+    )
+    (pin "1")
+  )
+  (symbol (lib_id "power:VCC") (at 40.64 77.47 90) (unit 1)
+    (in_bom yes) (on_board yes)
+    (property "Reference" "#PWR0142" (id 0) (at 44.45 77.47 0)
+      (effects (font (size 1.27 1.27)) hide)
+    )
+    (property "Value" "VCC" (id 1) (at 36.83 77.47 90)
+      (effects (font (size 1.27 1.27)) (justify left))
+    )
+    (property "Footprint" "" (id 2) (at 40.64 77.47 0)
+      (effects (font (size 1.27 1.27)) hide)
+    )
+    (property "Datasheet" "" (id 3) (at 40.64 77.47 0)
+      (effects (font (size 1.27 1.27)) hide)
+    )
+    (pin "1")
+  )
+  (symbol (lib_id "power:VS") (at 40.64 86.36 90) (unit 1)
+    (in_bom yes) (on_board yes)
+    (property "Reference" "#PWR0140" (id 0) (at 44.45 91.44 0)
+      (effects (font (size 1.27 1.27)) hide)
+    )
+    (property "Value" "VS" (id 1) (at 36.83 86.36 90)
+      (effects (font (size 1.27 1.27)) (justify left))
+    )
+    (property "Footprint" "" (id 2) (at 40.64 86.36 0)
+      (effects (font (size 1.27 1.27)) hide)
+    )
+    (property "Datasheet" "" (id 3) (at 40.64 86.36 0)
+      (effects (font (size 1.27 1.27)) hide)
+    )
+    (pin "1")
+  )
+  (symbol (lib_id "power:VCC") (at 40.64 88.9 90) (unit 1)
+    (in_bom yes) (on_board yes)
+    (property "Reference" "#PWR0141" (id 0) (at 44.45 88.9 0)
+      (effects (font (size 1.27 1.27)) hide)
+    )
+    (property "Value" "VCC" (id 1) (at 36.83 88.9 90)
+      (effects (font (size 1.27 1.27)) (justify left))
+    )
+    (property "Footprint" "" (id 2) (at 40.64 88.9 0)
+      (effects (font (size 1.27 1.27)) hide)
+    )
+    (property "Datasheet" "" (id 3) (at 40.64 88.9 0)
+      (effects (font (size 1.27 1.27)) hide)
+    )
+    (pin "1")
   )
   (symbol (lib_id "power:VCC") (at 107.95 85.09 90) (unit 1)
@@
     )
     (pin "1")
+  )
+  (symbol (lib_id "Device:R") (at 45.72 74.93 90) (unit 1)
+    (in_bom yes) (on_board yes)
+    (property "Reference" "R83" (id 0) (at 43.18 72.39 90)
+      (effects (font (size 1.27 1.27)) (justify left))
+    )
+    (property "Value" "0R (dnp)" (id 1) (at 53.34 72.39 90)
+      (effects (font (size 1.27 1.27)) (justify left))
+    )
+    (property "Footprint" "Resistor_SMD:R_0603_1608Metric" (id 2) (at 45.72 76.708 90)
+      (effects (font (size 1.27 1.27)) hide)
+    )
+    (property "Datasheet" "~" (id 3) (at 45.72 74.93 0)
+      (effects (font (size 1.27 1.27)) hide)
+    )
+    (pin "1")
+    (pin "2")
+  )
+  (symbol (lib_id "Device:R") (at 45.72 77.47 90) (unit 1)
+    (in_bom yes) (on_board yes)
+    (property "Reference" "R84" (id 0) (at 43.18 80.01 90)
+      (effects (font (size 1.27 1.27)) (justify left))
+    )
+    (property "Value" "0R (dnp)" (id 1) (at 53.34 80.01 90)
+      (effects (font (size 1.27 1.27)) (justify left))
+    )
+    (property "Footprint" "Resistor_SMD:R_0603_1608Metric" (id 2) (at 45.72 79.248 90)
+      (effects (font (size 1.27 1.27)) hide)
+    )
+    (property "Datasheet" "~" (id 3) (at 45.72 77.47 0)
+      (effects (font (size 1.27 1.27)) hide)
+    )
+    (pin "1")
+    (pin "2")
+  )
+  (symbol (lib_id "Device:R") (at 45.72 86.36 90) (unit 1)
+    (in_bom yes) (on_board yes)
+    (property "Reference" "R85" (id 0) (at 43.18 83.82 90)
+      (effects (font (size 1.27 1.27)) (justify left))
+    )
+    (property "Value" "0R (dnp)" (id 1) (at 53.34 83.82 90)
+      (effects (font (size 1.27 1.27)) (justify left))
+    )
+    (property "Footprint" "Resistor_SMD:R_0603_1608Metric" (id 2) (at 45.72 88.138 90)
+      (effects (font (size 1.27 1.27)) hide)
+    )
+    (property "Datasheet" "~" (id 3) (at 45.72 86.36 0)
+      (effects (font (size 1.27 1.27)) hide)
+    )
+    (pin "1")
+    (pin "2")
+  )
+  (symbol (lib_id "Device:R") (at 45.72 88.9 90) (unit 1)
+    (in_bom yes) (on_board yes)
+    (property "Reference" "R86" (id 0) (at 43.18 91.44 90)
+      (effects (font (size 1.27 1.27)) (justify left))
+    )
+    (property "Value" "0R (dnp)" (id 1) (at 53.34 91.44 90)
+      (effects (font (size 1.27 1.27)) (justify left))
+    )
+    (property "Footprint" "Resistor_SMD:R_0603_1608Metric" (id 2) (at 45.72 90.678 90)
+      (effects (font (size 1.27 1.27)) hide)
+    )
+    (property "Datasheet" "~" (id 3) (at 45.72 88.9 0)
+      (effects (font (size 1.27 1.27)) hide)
+    )
+    (pin "1")
+    (pin "2")
   )
   (symbol (lib_id "Device:R") (at 163.83 53.34 0) (unit 1)
@@
       (reference "#PWR0139") (unit 1) (value "GND") (footprint "")
     )
+    (path "/b57f8e28-7908-4723-badc-3fe03a3935fc"
+      (reference "#PWR0140") (unit 1) (value "VS") (footprint "")
+    )
+    (path "/ae4e67a3-9499-41c5-a7c6-18fc9d44f5b4"
+      (reference "#PWR0141") (unit 1) (value "VCC") (footprint "")
+    )
+    (path "/24f78540-75c5-4fef-a7dc-78513d9d1b78"
+      (reference "#PWR0142") (unit 1) (value "VCC") (footprint "")
+    )
+    (path "/d2559b76-149c-4da3-b5ef-16be5268b22f"
+      (reference "#PWR0143") (unit 1) (value "VS") (footprint "")
+    )
     (path "/e6f6539b-7042-4274-a151-2d1acf711eec/00a7c237-7ff9-409c-a59d-ed31d0075cb7"
       (reference "C1") (unit 1) (value "100n") (footprint "Capacitor_SMD:C_0603_1608Metric")
@@
       (reference "R82") (unit 1) (value "10k") (footprint "Resistor_SMD:R_0603_1608Metric")
     )
+    (path "/e63abd66-2f14-4693-aaf3-9cf3a3fbe563"
+      (reference "R83") (unit 1) (value "0R (dnp)") (footprint "Resistor_SMD:R_0603_1608Metric")
+    )
+    (path "/21b92d04-ecab-4a3a-b78f-24a87d0e89a6"
+      (reference "R84") (unit 1) (value "0R (dnp)") (footprint "Resistor_SMD:R_0603_1608Metric")
+    )
+    (path "/b1c21f1e-d629-4c17-aeda-516448128868"
+      (reference "R85") (unit 1) (value "0R (dnp)") (footprint "Resistor_SMD:R_0603_1608Metric")
+    )
+    (path "/94367be6-9cc9-4d68-bc55-06c5132b61cd"
+      (reference "R86") (unit 1) (value "0R (dnp)") (footprint "Resistor_SMD:R_0603_1608Metric")
+    )
     (path "/e6f6539b-7042-4274-a151-2d1acf711eec/90a1bdc2-1ee2-4aa1-834a-a7cf72c673be"

Commit message: moar woerk
Parts:
- added C10, C11, C13, C14: 100n, Capacitor_SMD:C_0603_1608Metric, symbol Device:C_Small
- added C12, C15: 10u, Capacitor_Tantalum_SMD:CP_EIA-3216-18_Kemet-A, symbol Device:C_Polarized_Small
- added D20: SOT23 A-C-K, Package_TO_SOT_SMD:SOT-23, symbol Device:D_Dual_Series_ACK_Parallel
- added D21: SS1P3L, Diode_SMD:D_SMF, symbol Device:D_Schottky_Small
- added D22, D23: LED, LED_SMD:LED_0603_1608Metric, symbol Device:LED
- added J3: Screw_Terminal_01x04, TerminalBlock_MetzConnect:TerminalBlock_MetzConnect_Type086_RT03404HBLC_1x04_P3.81mm_Horizontal, symbol Connector:Screw_Terminal_01x04
- added L1: L_Small, Inductor_SMD:L_Coilcraft_XxL4020, symbol Device:L_Small
- added R87, R88, R89: 68R, Resistor_SMD:R_0603_1608Metric, symbol Device:R
- added R91, R93, R96, R97, R98, R99: 10k, Resistor_SMD:R_0603_1608Metric, symbol Device:R
- added R92: 150k, Resistor_SMD:R_0603_1608Metric, symbol Device:R
- added R94, R95: 1k, Resistor_SMD:R_0603_1608Metric, symbol Device:R
- added U13: 74HCT244, Package_SO:SSOP-20_4.4x6.5mm_P0.65mm, symbol 74xx:74HCT244
- added U14: LM2734Y, Package_TO_SOT_SMD:TSOT-23-6, symbol Regulator_Switching:LM2734Y
Connections:
- net DI: now also R87.2; no longer J2.1 (Pin_1)
- net GND: now also C10.1, C11.1, C12.2, C14.1, C15.2, D21.2 (A), D22.1 (K), D23.1 (K), J3.2 (Pin_2), J3.4 (Pin_4), R93.1, R97.2, R98.2, R99.2, U13.1 (1OE), U13.10 (GND), U13.11 (2A3), U13.13 (2A2), U13.15 (2A1), U13.17 (2A0), U13.19 (2OE), U14.2 (GND)
- net LE: now also R88.2; no longer J2.3 (Pin_3)
- net SCK: now also R89.2; no longer J2.2 (Pin_2)
- net VCC: now also C10.2, C14.2, C15.1, D20.2 (A), J3.3 (Pin_3), L1.2, R92.1, R95.1, R96.1, U13.20 (VCC)
- net VS: now also C11.2, C12.1, J3.1 (Pin_1), R91.1, R94.1, U14.5 (VIN)
- net ~{ROW_OE}: now also U13.12 (1Y3); no longer J2.4 (Pin_4)
- new net: R89.1, U13.14 (1Y2)
- new net: R88.1, U13.16 (1Y1)
- new net: R87.1, U13.18 (1Y0)
- new net: R91.2, U14.4 (EN)
- new net: D22.2 (A), R94.2
- new net: D23.2 (A), R95.2
- new net DI_LV: J2.1 (Pin_1), R97.1, U13.2 (1A0)
- new net LE_LV: J2.3 (Pin_3), R98.1, U13.4 (1A1)
- new net SCK_LV: J2.2 (Pin_2), R99.1, U13.6 (1A2)
- new net VREG_BOOST: C13.2, D20.3 (K), U14.1 (BOOST)
- new net VREG_FB: R92.2, R93.2, U14.3 (FB)
- new net VREG_SW: C13.1, D21.1 (K), L1.1, U14.6 (SW)
- new net ~{ROW_OE}_LV: J2.4 (Pin_4), R96.2, U13.8 (1A3)
- no-connect marks 10 -> 15
Other:
- moved on the sheet: J2

Commit message: more work
Parts:
- removed C9: 100n, Capacitor_SMD:C_0603_1608Metric, symbol Device:C_Small
- removed U12: 74HCT595, Package_SO:SOIC-16_3.9x9.9mm_P1.27mm, symbol 74xx:74HCT595
- added J4: Conn_02x06_Odd_Even, Connector_IDC:IDC-Header_2x06_P2.54mm_Vertical, symbol Connector_Generic:Conn_02x06_Odd_Even
- added JP1, JP2, JP3, JP4, JP5, JP6: SolderJumper_2_Bridged, Jumper:SolderJumper-2_P1.3mm_Bridged_Pad1.0x1.5mm, symbol Jumper:SolderJumper_2_Bridged
- added R100, R101, R102, R103, R104, R90: 68R, Resistor_SMD:R_0603_1608Metric, symbol Device:R
- added R105, R106, R107, R108: 0R (dnp), Resistor_SMD:R_0603_1608Metric, symbol Device:R
- added U12: ULN2803A, Package_SO:SOIC-18W_7.5x11.6mm_P1.27mm, symbol Transistor_Array:ULN2803A
Connections:
- net COL_A0: now also U12.11 (O8); no longer U11.15 (QA)
- net COL_A1: now also U12.12 (O7); no longer U11.1 (QB)
- net COL_A2: now also U12.13 (O6); no longer U11.2 (QC)
- net COL_B0: now also U12.14 (O5); no longer U11.3 (QD)
- net COL_B1: now also U12.15 (O4); no longer U11.4 (QE)
- net COL_D: now also U12.16 (O3); no longer U10.1 (A), U11.5 (QF)
- net DI: now also R89.2, U11.14 (SER); no longer R87.2
- net DI_LV: now also R99.1, U13.6 (1A2); no longer R97.1, U13.2 (1A0)
- net GND: now also J4.10 (Pin_10), J4.9 (Pin_9), JP1.2 (B), JP2.2 (B), JP3.2 (B), JP4.2 (B), JP5.2 (B), JP6.2 (B), U12.9 (GND); no longer U13.11 (2A3), U13.13 (2A2), U13.15 (2A1), U13.17 (2A0)
- net LE: now also U13.15 (2A1)
- net MODULE_A0: now also U12.17 (O2)
- net MODULE_A1: now also U12.18 (O1)
- net MODULE_A2: now also JP1.1 (A)
- net MODULE_A3: now also JP2.1 (A)
- net MODULE_A4: now also JP3.1 (A)
- net MODULE_A5: now also JP4.1 (A)
- net MODULE_A6: now also JP5.1 (A)
- net MODULE_A7: now also JP6.1 (A)
- net SCK: now also R87.2, U13.17 (2A0); no longer R89.2
- net SCK_LV: now also R97.1, U13.2 (1A0); no longer R99.1, U13.6 (1A2)
- net VCC: now also R107.2
- net VREG_BOOST: no longer C13.2, D20.3 (K), U14.1 (BOOST)
- net VS: now also U12.10 (COM)
- net ~{ROW_N_OE}: now also R90.2; no longer U10.4 (Y1)
- net ~{ROW_OE}: now also U13.11 (2A3)
- net ~{ROW_P_OE}: now also R100.2; no longer U10.6 (Y0)
- net at U11.6 (QG): now also U12.2 (I2)
- net at U11.7 (QH): now also U12.1 (I1)
- net DI_x: now reaches R89.1, U13.14 (1Y2)
- net DI_x: now also R105.1
- net at U13.3 (2Y0): now also R101.1
- net at U13.5 (2Y1): now also R102.1
- net at U13.7 (2Y2): now also R103.1
- net at U13.9 (2Y3): now also R104.1
- net at J2.11 (Pin_11): now also J2.12 (Pin_12), J4.11 (Pin_11), J4.12 (Pin_12), R107.1
- net at J2.5 (Pin_5): now also R108.1
- new net: C13.2, D20.3 (K)
- new net: R100.1, U10.4 (Y1)
- new net: U11.1 (QB), U12.7 (I7)
- new net: U11.15 (QA), U12.8 (I8)
- new net: U11.2 (QC), U12.6 (I6)
- new net: U11.3 (QD), U12.5 (I5)
- new net: U11.4 (QE), U12.4 (I4)
- new net: R90.1, U10.6 (Y0)
- new net COL_D_LV: U10.1 (A), U11.5 (QF), U12.3 (I3)
- new net DO: J4.1 (Pin_1), R103.2, R108.2
- new net DO_LV_SEL: R105.2, R106.2, U13.13 (2A2)
- new net DO_P: R106.1
- new net LE_OUT: J4.3 (Pin_3), R102.2
- new net SCK_OUT: J4.2 (Pin_2), R101.2
- new net ~{ROW_OE}_OUT: J4.4 (Pin_4), R104.2
- no-connect marks 15 -> 10
Other:
- sheet Row Drivers Negative ports: added ROW_N_DO; removed none
- sheet Row Drivers Positive ports: added ROW_P_DO; removed none
- note added: "COL_D_LV=H, COL_D=L"
- note added: "COL_D_LV=L, COL_D=H"
- note removed: "COL_D=H"
- note removed: "COL_D=L"
- moved on the sheet: C10, C7, C8, J2, R79, R80, R81, R87, R88, R89, R96, R97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

Commit message: More work, moved digital stuff to sub-schematic.
Parts:
- removed C7, C8: 100n, Capacitor_SMD:C_0603_1608Metric, symbol Device:C_Small
- removed R100, R90: 68R, Resistor_SMD:R_0603_1608Metric, symbol Device:R
- removed R80, R81, R82: 10k, Resistor_SMD:R_0603_1608Metric, symbol Device:R
- removed U10: 74LVC1G19, Package_TO_SOT_SMD:SOT-563, symbol 74xGxx:74LVC1G19
- removed U11: 74HCT595, Package_SO:SOIC-16_3.9x9.9mm_P1.27mm, symbol 74xx:74HCT595
- removed U12: ULN2803A, Package_SO:SOIC-18W_7.5x11.6mm_P1.27mm, symbol Transistor_Array:ULN2803A
- added C16, C18: 10u, Capacitor_Tantalum_SMD:CP_EIA-3216-18_Kemet-A, symbol Device:C_Polarized_Small
- added C17, C9: 100n, Capacitor_SMD:C_0603_1608Metric, symbol Device:C_Small
- added D24: LED, LED_SMD:LED_0603_1608Metric, symbol Device:LED
- added U15: AP1117-33, Package_TO_SOT_SMD:SOT-223-3_TabPin2, symbol Regulator_Linear:AP1117-33
- R79: value 10k -> 1k
Connections:
- net GND: now also C16.2, C17.1, C18.2, C9.1, D24.1 (K), U15.1 (GND); no longer R79.2
- net LE: no longer R79.1
- net VCC: now also C16.1, C9.2, U15.3 (VI)
- net VREG_BOOST: now also C13.2, D20.3 (K), U14.1 (BOOST)
- new net: D24.2 (A), R79.2
- new net +3V3: C17.2, C18.1, R79.1, U15.2 (VO)
Other:
- added sheet Digital Pin Drivers (drv_digital.kicad_sch)
- note added: "Input"
- note added: "Output (potentially to chain)"
- note removed: "COL_D_LV=H, COL_D=L"
- note removed: "COL_D_LV=L, COL_D=H"
- note removed: "~{E}=H, A=X → Y0=H, Y1=H ~{E}=L, A=H → Y0=H, Y1=L ~{E}=L, A=L → Y0=L, Y1=H"
- moved on the sheet: C10, C11, C12, C13, C14, C15, D20, D21, D22, D23, J2, J3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
